Commit message: feat: Robot model redesign
Adjust size of chassis and wheels. Remove caster wheels.

File: rover/urdf/rover.xacro (robot description, xacro)
@@ -22,5 +22,5 @@
       <origin xyz="0 0 0" rpy=" 0 0 0"/>
       <geometry>
-        <box size=".4 .2 .1"/>
+        <box size=".46 .2 .1"/>
       </geometry>
     </collision>
@@ -28,51 +28,7 @@
       <origin xyz="0 0 0" rpy=" 0 0 0"/>
       <geometry>
-        <box size=".4 .2 .1"/>
+        <box size=".46 .2 .1"/>
       </geometry>
       <material name="black"/>
-    </visual>
-    <collision name='back_caster_collision'>
-      <origin xyz="-0.15 0 -0.05" rpy=" 0 0 0"/>
-      <geometry>
-        <sphere radius="0.05"/>
-      </geometry>
-      <surface>
-        <friction>
-          <ode>
-            <mu>0</mu>
-            <mu2>0</mu2>
-            <slip1>1.0</slip1>
-            <slip2>1.0</slip2>
-          </ode>
-        </friction>
-      </surface>
-    </collision>
-    <visual name='back_caster_visual'>
-      <origin xyz="-0.15 0 -0.05" rpy=" 0 0 0"/>
-      <geometry>
-        <sphere radius="0.05"/>
-      </geometry>
-    </visual>
-    <collision name='front_caster_collision'>
-      <origin xyz="0.15 0 -0.05" rpy=" 0 0 0"/>
-      <geometry>
-        <sphere radius="0.05"/>
-      </geometry>
-      <surface>
-        <friction>
-          <ode>
-            <mu>0</mu>
-            <mu2>0</mu2>
-            <slip1>1.0</slip1>
-            <slip2>1.0</slip2>
-          </ode>
-        </friction>
-      </surface>
-    </collision>
-    <visual name='front_caster_visual'>
-      <origin xyz="0.15 0 -0.05" rpy=" 0 0 0"/>
-      <geometry>
-        <sphere radius="0.05"/>
-      </geometry>
     </visual>
   </link>
@@ -91,5 +47,5 @@
       <origin xyz="0 0 0" rpy=" 0 1.5707 1.5707"/>
       <geometry>
-        <cylinder length="0.05" radius="0.1"/>
+        <cylinder length="0.056" radius="0.084"/>
       </geometry>
     </collision>
@@ -97,5 +53,5 @@
       <origin xyz="0 0 0" rpy=" 0 1.5707 1.5707"/>
       <geometry>
-        <cylinder length="0.05" radius="0.1"/>
+        <cylinder length="0.056" radius="0.084"/>
       </geometry>
     </visual>
@@ -123,5 +79,5 @@
       <origin xyz="0 0 0" rpy=" 0 1.5707 1.5707"/>
       <geometry>
-        <cylinder length="0.05" radius="0.1"/>
+        <cylinder length="0.056" radius="0.084"/>
       </geometry>
     </collision>
@@ -129,5 +85,5 @@
       <origin xyz="0 0 0" rpy=" 0 1.5707 1.5707"/>
       <geometry>
-        <cylinder length="0.05" radius="0.1"/>
+        <cylinder length="0.056" radius="0.084"/>
       </geometry>
     </visual>

Commit message: fix: Adjust joint origin x for camera and hokuyo

File: rover/urdf/rover.xacro (robot description, xacro)
@@ -123,5 +123,5 @@
   </link>
   <joint type="fixed" name="camera_joint">
-    <origin xyz="0.2 0 0" rpy="0 0 0"/>
+    <origin xyz="0.23 0 0" rpy="0 0 0"/>
     <child link="camera"/>
     <parent link="chassis"/>
@@ -156,5 +156,5 @@
   </link>
   <joint type="fixed" name="hokuyo_joint">
-    <origin xyz=".15 0 .1" rpy="0 0 0"/>
+    <origin xyz=".2 0 .1" rpy="0 0 0"/>
     <child link="hokuyo"/>
     <parent link="chassis"/>

Commit message: feat: Move wheels to the front

File: rover/urdf/rover.xacro (robot description, xacro)
@@ -33,5 +33,6 @@
     </visual>
   </link>
-  <link name='left_wheel'>
+  <!-- front wheels -->
+  <link name='front_left_wheel'>
     <pose>0 0 0.1 0 0 0</pose>
     <inertial>
@@ -44,5 +45,5 @@
       />
     </inertial>
-    <collision name='left_wheel_collision'>
+    <collision name='front_left_wheel_collision'>
       <origin xyz="0 0 0" rpy=" 0 1.5707 1.5707"/>
       <geometry>
@@ -50,5 +51,5 @@
       </geometry>
     </collision>
-    <visual name='left_wheel_visual'>
+    <visual name='front_left_wheel_visual'>
       <origin xyz="0 0 0" rpy=" 0 1.5707 1.5707"/>
       <geometry>
@@ -57,7 +58,7 @@
     </visual>
   </link>
-  <joint type="continuous" name="left_wheel_hinge">
-    <origin xyz="0 0.15 0" rpy="0 0 0"/>
-    <child link="left_wheel"/>
+  <joint type="continuous" name="front_left_wheel_hinge">
+    <origin xyz="0.15 0.15 0" rpy="0 0 0"/>
+    <child link="front_left_wheel"/>
     <parent link="chassis"/>
     <axis xyz="0 1 0" rpy="0 0 0"/>
@@ -65,5 +66,5 @@
     <joint_properties damping="1.0" friction="1.0"/>
   </joint>
-  <link name='right_wheel'>
+  <link name='front_right_wheel'>
     <pose>0 0 0.1 0 0 0</pose>
     <inertial>
@@ -76,5 +77,5 @@
       />
     </inertial>
-    <collision name='right_wheel_collision'>
+    <collision name='front_right_wheel_collision'>
       <origin xyz="0 0 0" rpy=" 0 1.5707 1.5707"/>
       <geometry>
@@ -82,5 +83,5 @@
       </geometry>
     </collision>
-    <visual name='right_wheel_visual'>
+    <visual name='front_right_wheel_visual'>
       <origin xyz="0 0 0" rpy=" 0 1.5707 1.5707"/>
       <geometry>
@@ -89,7 +90,7 @@
     </visual>
   </link>
-  <joint type="continuous" name="right_wheel_hinge">
-    <origin xyz="0 -0.15 0" rpy="0 0 0"/>
-    <child link="right_wheel"/>
+  <joint type="continuous" name="front_right_wheel_hinge">
+    <origin xyz="0.15 -0.15 0" rpy="0 0 0"/>
+    <child link="front_right_wheel"/>
     <parent link="chassis"/>
     <axis xyz="0 1 0" rpy="0 0 0"/>

Commit message: feat: Add rear wheels

File: rover/urdf/rover.xacro (robot description, xacro)
@@ -164,3 +164,68 @@
     <joint_properties damping="1.0" friction="1.0"/>
   </joint>
+  <!-- rear wheels -->
+  <link name='rear_left_wheel'>
+    <pose>0 0 0.1 0 0 0</pose>
+    <inertial>
+      <mass value="5.0"/>
+      <origin xyz="0 0 0" rpy=" 0 1.5707 1.5707"/>
+      <inertia
+          ixx="0.1" ixy="0" ixz="0"
+          iyy="0.1" iyz="0"
+          izz="0.1"
+      />
+    </inertial>
+    <collision name='rear_left_wheel_collision'>
+      <origin xyz="0 0 0" rpy=" 0 1.5707 1.5707"/>
+      <geometry>
+        <cylinder length="0.056" radius="0.084"/>
+      </geometry>
+    </collision>
+    <visual name='rear_left_wheel_visual'>
+      <origin xyz="0 0 0" rpy=" 0 1.5707 1.5707"/>
+      <geometry>
+        <cylinder length="0.056" radius="0.084"/>
+      </geometry>
+    </visual>
+  </link>
+  <joint type="continuous" name="rear_left_wheel_hinge">
+    <origin xyz="-0.15 0.15 0" rpy="0 0 0"/>
+    <child link="rear_left_wheel"/>
+    <parent link="chassis"/>
+    <axis xyz="0 1 0" rpy="0 0 0"/>
+    <limit effort="10000" velocity="1000"/>
+    <joint_properties damping="1.0" friction="1.0"/>
+  </joint>
+  <link name='rear_right_wheel'>
+    <pose>0 0 0.1 0 0 0</pose>
+    <inertial>
+      <mass value="5.0"/>
+      <origin xyz="0 0 0" rpy=" 0 1.5707 1.5707"/>
+      <inertia
+          ixx="0.1" ixy="0" ixz="0"
+          iyy="0.1" iyz="0"
+          izz="0.1"
+      />
+    </inertial>
+    <collision name='rear_right_wheel_collision'>
+      <origin xyz="0 0 0" rpy=" 0 1.5707 1.5707"/>
+      <geometry>
+        <cylinder length="0.056" radius="0.084"/>
+      </geometry>
+    </collision>
+    <visual name='rear_right_wheel_visual'>
+      <origin xyz="0 0 0" rpy=" 0 1.5707 1.5707"/>
+      <geometry>
+        <cylinder length="0.056" radius="0.084"/>
+      </geometry>
+    </visual>
+  </link>
+  <joint type="continuous" name="rear_right_wheel_hinge">
+    <origin xyz="-0.15 -0.15 0" rpy="0 0 0"/>
+    <child link="rear_right_wheel"/>
+    <parent link="chassis"/>
+    <axis xyz="0 1 0" rpy="0 0 0"/>
+    <limit effort="10000" velocity="1000"/>
+    <joint_properties damping="1.0" friction="1.0"/>
+  </joint>
 </robot>

Commit message: feat: Replace rear wheels by caster

File: rover/urdf/rover.xacro (robot description, xacro)
@@ -31,4 +31,26 @@
       </geometry>
       <material name="black"/>
+    </visual>
+    <collision name='back_caster_collision'>
+      <origin xyz="-0.18 0 -0.042" rpy=" 0 0 0"/>
+      <geometry>
+        <sphere radius="0.042"/>
+      </geometry>
+      <surface>
+        <friction>
+          <ode>
+            <mu>0</mu>
+            <mu2>0</mu2>
+            <slip1>1.0</slip1>
+            <slip2>1.0</slip2>
+          </ode>
+        </friction>
+      </surface>
+    </collision>
+    <visual name='back_caster_visual'>
+      <origin xyz="-0.18 0 -0.042" rpy=" 0 0 0"/>
+      <geometry>
+        <sphere radius="0.042"/>
+      </geometry>
     </visual>
   </link>
@@ -164,68 +186,3 @@
     <joint_properties damping="1.0" friction="1.0"/>
   </joint>
-  <!-- rear wheels -->
-  <link name='rear_left_wheel'>
-    <pose>0 0 0.1 0 0 0</pose>
-    <inertial>
-      <mass value="5.0"/>
-      <origin xyz="0 0 0" rpy=" 0 1.5707 1.5707"/>
-      <inertia
-          ixx="0.1" ixy="0" ixz="0"
-          iyy="0.1" iyz="0"
-          izz="0.1"
-      />
-    </inertial>
-    <collision name='rear_left_wheel_collision'>
-      <origin xyz="0 0 0" rpy=" 0 1.5707 1.5707"/>
-      <geometry>
-        <cylinder length="0.056" radius="0.084"/>
-      </geometry>
-    </collision>
-    <visual name='rear_left_wheel_visual'>
-      <origin xyz="0 0 0" rpy=" 0 1.5707 1.5707"/>
-      <geometry>
-        <cylinder length="0.056" radius="0.084"/>
-      </geometry>
-    </visual>
-  </link>
-  <joint type="continuous" name="rear_left_wheel_hinge">
-    <origin xyz="-0.15 0.15 0" rpy="0 0 0"/>
-    <child link="rear_left_wheel"/>
-    <parent link="chassis"/>
-    <axis xyz="0 1 0" rpy="0 0 0"/>
-    <limit effort="10000" velocity="1000"/>
-    <joint_properties damping="1.0" friction="1.0"/>
-  </joint>
-  <link name='rear_right_wheel'>
-    <pose>0 0 0.1 0 0 0</pose>
-    <inertial>
-      <mass value="5.0"/>
-      <origin xyz="0 0 0" rpy=" 0 1.5707 1.5707"/>
-      <inertia
-          ixx="0.1" ixy="0" ixz="0"
-          iyy="0.1" iyz="0"
-          izz="0.1"
-      />
-    </inertial>
-    <collision name='rear_right_wheel_collision'>
-      <origin xyz="0 0 0" rpy=" 0 1.5707 1.5707"/>
-      <geometry>
-        <cylinder length="0.056" radius="0.084"/>
-      </geometry>
-    </collision>
-    <visual name='rear_right_wheel_visual'>
-      <origin xyz="0 0 0" rpy=" 0 1.5707 1.5707"/>
-      <geometry>
-        <cylinder length="0.056" radius="0.084"/>
-      </geometry>
-    </visual>
-  </link>
-  <joint type="continuous" name="rear_right_wheel_hinge">
-    <origin xyz="-0.15 -0.15 0" rpy="0 0 0"/>
-    <child link="rear_right_wheel"/>
-    <parent link="chassis"/>
-    <axis xyz="0 1 0" rpy="0 0 0"/>
-    <limit effort="10000" velocity="1000"/>
-    <joint_properties damping="1.0" friction="1.0"/>
-  </joint>
 </robot>

Commit message: feat: Make chassis smaller and adjust joints

File: rover/urdf/rover.xacro (robot description, xacro)
@@ -22,5 +22,5 @@
       <origin xyz="0 0 0" rpy=" 0 0 0"/>
       <geometry>
-        <box size=".46 .2 .1"/>
+        <box size=".38 .2 .1"/>
       </geometry>
     </collision>
@@ -28,10 +28,10 @@
       <origin xyz="0 0 0" rpy=" 0 0 0"/>
       <geometry>
-        <box size=".46 .2 .1"/>
+        <box size=".38 .2 .1"/>
       </geometry>
       <material name="black"/>
     </visual>
     <collision name='back_caster_collision'>
-      <origin xyz="-0.18 0 -0.042" rpy=" 0 0 0"/>
+      <origin xyz="-0.14 0 -0.042" rpy=" 0 0 0"/>
       <geometry>
         <sphere radius="0.042"/>
@@ -49,5 +49,5 @@
     </collision>
     <visual name='back_caster_visual'>
-      <origin xyz="-0.18 0 -0.042" rpy=" 0 0 0"/>
+      <origin xyz="-0.14 0 -0.042" rpy=" 0 0 0"/>
       <geometry>
         <sphere radius="0.042"/>
@@ -81,5 +81,5 @@
   </link>
   <joint type="continuous" name="front_left_wheel_hinge">
-    <origin xyz="0.15 0.15 0" rpy="0 0 0"/>
+    <origin xyz="0.12 0.15 0" rpy="0 0 0"/>
     <child link="front_left_wheel"/>
     <parent link="chassis"/>
@@ -113,5 +113,5 @@
   </link>
   <joint type="continuous" name="front_right_wheel_hinge">
-    <origin xyz="0.15 -0.15 0" rpy="0 0 0"/>
+    <origin xyz="0.12 -0.15 0" rpy="0 0 0"/>
     <child link="front_right_wheel"/>
     <parent link="chassis"/>
@@ -146,5 +146,5 @@
   </link>
   <joint type="fixed" name="camera_joint">
-    <origin xyz="0.23 0 0" rpy="0 0 0"/>
+    <origin xyz="0.21 0 0" rpy="0 0 0"/>
     <child link="camera"/>
     <parent link="chassis"/>
@@ -179,5 +179,5 @@
   </link>
   <joint type="fixed" name="hokuyo_joint">
-    <origin xyz=".2 0 .1" rpy="0 0 0"/>
+    <origin xyz="0.14 0.0 0.084" rpy="0 0 0"/>
     <child link="hokuyo"/>
     <parent link="chassis"/>

Commit message: feat: Customize link colors

File: rover/urdf/rover.xacro (robot description, xacro)
@@ -2,4 +2,13 @@
 <robot name="rover" xmlns:xacro="http://www.ros.org/wiki/xacro">
   <xacro:include filename="$(find rover)/urdf/rover.gazebo" />
+  <material name="skyblue">
+    <color rgba="0.13 0.44 0.70 1.0"/>
+  </material>
+  <material name="white">
+    <color rgba="1.0 1.0 1.0 1.0"/>
+  </material>
+  <material name="orange">
+    <color rgba="${255/255} ${108/255} ${10/255} 1.0"/>
+  </material>
   <link name="robot_footprint"></link>
   <joint name="robot_footprint_joint" type="fixed">
@@ -30,5 +39,5 @@
         <box size=".38 .2 .1"/>
       </geometry>
-      <material name="black"/>
+      <material name="white"/>
     </visual>
     <collision name='back_caster_collision'>
@@ -75,4 +84,5 @@
     <visual name='front_left_wheel_visual'>
       <origin xyz="0 0 0" rpy=" 0 1.5707 1.5707"/>
+      <material name="orange"/>
       <geometry>
         <cylinder length="0.056" radius="0.084"/>
@@ -107,4 +117,5 @@
     <visual name='front_right_wheel_visual'>
       <origin xyz="0 0 0" rpy=" 0 1.5707 1.5707"/>
+      <material name="orange"/>
       <geometry>
         <cylinder length="0.056" radius="0.084"/>
@@ -140,4 +151,5 @@
     <visual name='camera_visual'>
       <origin xyz="0 0 0" rpy=" 0 0 0"/>
+      <material name="skyblue"/>
       <geometry>
         <box size=".05 .05 .05"/>

Commit message: feat: Create custom rover version 3

File: rover/urdf/rover.xacro (robot description, xacro)
@@ -28,19 +28,93 @@
       />
     </inertial>
-    <collision name='collision'>
-      <origin xyz="0 0 0" rpy=" 0 0 0"/>
-      <geometry>
-        <box size=".38 .2 .1"/>
-      </geometry>
-    </collision>
-    <visual name='chassis_visual'>
-      <origin xyz="0 0 0" rpy=" 0 0 0"/>
-      <geometry>
-        <box size=".38 .2 .1"/>
+    <collision name='base_collision'>
+      <origin xyz="0 0 0" rpy=" 0 0 0"/>
+      <geometry>
+        <box size="0.38 0.1 0.1"/>
+      </geometry>
+    </collision>
+    <visual name='base_visual'>
+      <origin xyz="0 0 0" rpy=" 0 0 0"/>
+      <geometry>
+        <box size="0.38 0.1 0.1"/>
       </geometry>
       <material name="white"/>
     </visual>
-    <collision name='back_caster_collision'>
-      <origin xyz="-0.14 0 -0.042" rpy=" 0 0 0"/>
+    <collision name='left_wing_collision'>
+      <origin xyz="0 0.075 0" rpy=" 0 0 0"/>
+      <geometry>
+        <box size="0.28 0.05 0.1"/>
+      </geometry>
+    </collision>
+    <visual name='left_wing_visual'>
+      <origin xyz="0 0.075 0" rpy=" 0 0 0"/>
+      <geometry>
+        <box size="0.28 0.05 0.1"/>
+      </geometry>
+      <material name="white"/>
+    </visual>
+    <collision name='right_wing_collision'>
+      <origin xyz="0 -0.075 0" rpy=" 0 0 0"/>
+      <geometry>
+        <box size="0.28 0.05 0.1"/>
+      </geometry>
+    </collision>
+    <visual name='right_wing_visual'>
+      <origin xyz="0 -0.075 0" rpy=" 0 0 0"/>
+      <geometry>
+        <box size="0.28 0.05 0.1"/>
+      </geometry>
+      <material name="white"/>
+    </visual>
+    <collision name='front_left_fender_collision'>
+      <origin xyz="0.14 0.05 0" rpy="0 0 1.5707"/>
+      <geometry>
+        <cylinder length="0.1" radius="0.05"/>
+      </geometry>
+    </collision>
+    <visual name='front_left_fender_visual'>
+      <origin xyz="0.14 0.05 0" rpy="0 0 1.5707"/>
+      <geometry>
+        <cylinder length="0.1" radius="0.05"/>
+      </geometry>
+    </visual>
+    <collision name='front_right_fender_collision'>
+      <origin xyz="0.14 -0.05 0" rpy="0 0 1.5707"/>
+      <geometry>
+        <cylinder length="0.1" radius="0.05"/>
+      </geometry>
+    </collision>
+    <visual name='front_right_fender_visual'>
+      <origin xyz="0.14 -0.05 0" rpy="0 0 1.5707"/>
+      <geometry>
+        <cylinder length="0.1" radius="0.05"/>
+      </geometry>
+    </visual>
+    <collision name='rear_right_fender_collision'>
+      <origin xyz="-0.14 -0.05 0" rpy="0 0 1.5707"/>
+      <geometry>
+        <cylinder length="0.1" radius="0.05"/>
+      </geometry>
+    </collision>
+    <visual name='rear_right_fender_visual'>
+      <origin xyz="-0.14 -0.05 0" rpy="0 0 1.5707"/>
+      <geometry>
+        <cylinder length="0.1" radius="0.05"/>
+      </geometry>
+    </visual>
+    <collision name='rear_left_fender_collision'>
+      <origin xyz="-0.14 0.05 0" rpy="0 0 1.5707"/>
+      <geometry>
+        <cylinder length="0.1" radius="0.05"/>
+      </geometry>
+    </collision>
+    <visual name='rear_left_fender_visual'>
+      <origin xyz="-0.14 0.05 0" rpy="0 0 1.5707"/>
+      <geometry>
+        <cylinder length="0.1" radius="0.05"/>
+      </geometry>
+    </visual>
+    <collision name='front_caster_collision'>
+      <origin xyz="0.14 0 -0.042" rpy=" 0 0 0"/>
       <geometry>
         <sphere radius="0.042"/>
@@ -57,4 +131,26 @@
       </surface>
     </collision>
+    <visual name='front_caster_visual'>
+      <origin xyz="0.14 0 -0.042" rpy=" 0 0 0"/>
+      <geometry>
+        <sphere radius="0.042"/>
+      </geometry>
+    </visual>
+    <collision name='back_caster_collision'>
+      <origin xyz="-0.14 0 -0.042" rpy=" 0 0 0"/>
+      <geometry>
+        <sphere radius="0.042"/>
+      </geometry>
+      <surface>
+        <friction>
+          <ode>
+            <mu>0</mu>
+            <mu2>0</mu2>
+            <slip1>1.0</slip1>
+            <slip2>1.0</slip2>
+          </ode>
+        </friction>
+      </surface>
+    </collision>
     <visual name='back_caster_visual'>
       <origin xyz="-0.14 0 -0.042" rpy=" 0 0 0"/>
@@ -91,5 +187,5 @@
   </link>
   <joint type="continuous" name="front_left_wheel_hinge">
-    <origin xyz="0.12 0.15 0" rpy="0 0 0"/>
+    <origin xyz="0 0.15 0" rpy="0 0 0"/>
     <child link="front_left_wheel"/>
     <parent link="chassis"/>
@@ -124,5 +220,5 @@
   </link>
   <joint type="continuous" name="front_right_wheel_hinge">
-    <origin xyz="0.12 -0.15 0" rpy="0 0 0"/>
+    <origin xyz="0 -0.15 0" rpy="0 0 0"/>
     <child link="front_right_wheel"/>
     <parent link="chassis"/>
